File: cm3_audio.brd (EAGLE design)
At the start: 103 x 108.4 mm, 112 parts, among them IC1 PESD3V3L5UYSOT363, IC15 SN65220, IC2 AP2331W, IC4 MIC5205, IC5 TVS-DUAL-BI, IC6 TVS-DUAL-BI, IC7 WM8731WIDE, IC8 TVS-DUAL-BI, IC9 MAX98306ETD+T, J1 STEREO_HEADPHONE_NO_SWITCH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

Commit message: fixing codec layout
Parts:
- removed R46: 10k, osborn:0603-RES
- added C4: 100n, osborn:0603-CAP
- moved R10 91.7 mm to (111.7, 65.4)
- moved R9 91.7 mm to (111.7, 63.9)
- moved R11 22.2 mm to (18.6, 48.2), turned to 90 degrees
- moved R18 22.1 mm to (16.8, 44.8), turned to 90 degrees
- moved C53 21.8 mm to (24.0, 25.8), turned to 0 degrees
- moved R43 21.8 mm to (39.5, 28.3), turned to 90 degrees
- moved C63 20.3 mm to (41.3, 28.3), turned to 90 degrees
- moved C64 19.1 mm to (43.2, 28.4), turned to 270 degrees
- moved R45 19.1 mm to (47.1, 28.4), turned to 270 degrees
- moved C56 19.0 mm to (15.2, 29.1)
- moved R22 19.0 mm to (14.6, 23.8)
- moved JP8 18.8 mm to (52.7, 29.4), turned to 270 degrees
- moved C51 18.2 mm to (31.1, 26.4), turned to 0 degrees
- moved R44 18.1 mm to (45.2, 28.4), turned to 270 degrees
- moved C52 18.0 mm to (24.1, 28.9), turned to 180 degrees
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Connections:
- removed net N$56: IC7.22, R46.1
- net CM_BCLK: no longer JP2.6
- net CM_DIN: no longer JP2.8
- net CM_DOUT: no longer JP2.9
- net CM_LRCIN: no longer JP2.7
- net GND: now also C4.2, IC7.22
- net VCC_3V3: now also C4.1; no longer R46.2
Routing:
- net VCC_3V3: track 416.6 -> 232.1 mm, vias 5 -> 1
- net CM_LRCIN: track 124.1 -> 0.00 mm, vias 1 -> 0
- net CM_DOUT: track 123.2 -> 0.00 mm, vias 1 -> 0
- net CM_BCLK: track 120.9 -> 0.00 mm, vias 1 -> 0
- net CM_SCL: track 110.7 -> 0.00 mm, vias 1 -> 0
- net CM_SDA: track 110.5 -> 0.00 mm, vias 1 -> 0
- net VCC_5V: track 379.5 -> 278.2 mm
- net DIN: track 79.2 -> 0.00 mm
- net N$55: track 48.2 -> 0.00 mm
- net CM_DIN: track 46.9 -> 0.00 mm, vias 1 -> 0
- net N$53: track 35.6 -> 0.12 mm
- net RHPOUT: track 35.1 -> 6.44 mm
- net N$52: track 26.2 -> 0.04 mm
- net AVCC_3V3: track 59.0 -> 33.5 mm
- net N$51: track 23.9 -> 0.19 mm
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- added copper zone on layer 2, net GND
